Commit message: Experiment with removing namespace

File: urdf/little_helper10_arm_on_left.urdf (robot description, URDF)
Before this commit: robot little_helper10, 31 links, 30 joints
Links:
- removed link ur5_arm_1_base
- removed link ur5_arm_1_base_link
- removed link ur5_arm_1_base_link_inertia
- removed link ur5_arm_1_flange
- removed link ur5_arm_1_forearm_link
- removed link ur5_arm_1_shoulder_link
- removed link ur5_arm_1_tool0
- removed link ur5_arm_1_upper_arm_link
- removed link ur5_arm_1_wrist_1_link
- removed link ur5_arm_1_wrist_2_link
- removed link ur5_arm_1_wrist_3_link
- added link base
- added link base_link_inertia, mass 4.0; collision mesh filename=package://little_helper_urdf/ur5_to_convert/base.stl; visual mesh filename=package://little_helper_urdf/ur5_to_convert/base.dae
- added link flange
- added link forearm_link, mass 2.275; collision mesh filename=package://little_helper_urdf/ur5_to_convert/forearm.stl; visual mesh filename=package://little_helper_urdf/ur5_to_convert/forearm.dae
- added link shoulder_link, mass 3.7; collision mesh filename=package://little_helper_urdf/ur5_to_convert/shoulder.stl; visual mesh filename=package://little_helper_urdf/ur5_to_convert/shoulder.dae
- added link tool0
- added link upper_arm_link, mass 8.393; collision mesh filename=package://little_helper_urdf/ur5_to_convert/upperarm.stl; visual mesh filename=package://little_helper_urdf/ur5_to_convert/upperarm.dae
- added link wrist_1_link, mass 1.219; collision mesh filename=package://little_helper_urdf/ur5_to_convert/wrist1.stl; visual mesh filename=package://little_helper_urdf/ur5_to_convert/wrist1.dae
- added link wrist_2_link, mass 1.219; collision mesh filename=package://little_helper_urdf/ur5_to_convert/wrist2.stl; visual mesh filename=package://little_helper_urdf/ur5_to_convert/wrist2.dae
- added link wrist_3_link, mass 0.1879; collision mesh filename=package://little_helper_urdf/ur5_to_convert/wrist3.stl; visual mesh filename=package://little_helper_urdf/ur5_to_convert/wrist3.dae
- link base_link: mass 77.0 -> None; geometry 
Joints:
- removed joint ur5_arm_1_base_joint
- removed joint ur5_arm_1_base_link-base_fixed_joint
- removed joint ur5_arm_1_base_link-base_link_inertia
- removed joint ur5_arm_1_elbow_joint
- removed joint ur5_arm_1_flange-tool0
- removed joint ur5_arm_1_shoulder_lift_joint
- removed joint ur5_arm_1_shoulder_pan_joint
- removed joint ur5_arm_1_wrist_1_joint
- removed joint ur5_arm_1_wrist_2_joint
- removed joint ur5_arm_1_wrist_3-flange
- removed joint ur5_arm_1_wrist_3_joint
- added joint base_link-base_fixed_joint: type fixed, parent base_link, child base, origin xyz=0 0 0 rpy=0 0 3.14159265359
- added joint base_link-base_link_inertia: type fixed, parent base_link, child base_link_inertia, origin xyz=0 0 0 rpy=0 0 3.14159265359
- added joint elbow_joint: type revolute, parent upper_arm_link, child forearm_link, origin xyz=-0.425 0 0 rpy=0 0 0, axis 0 0 1, limit lower=-3.14159265359 upper=3.14159265359 effort=150.0 velocity=3.14159265359
- added joint flange-tool0: type fixed, parent flange, child tool0, origin xyz=0 0 0 rpy=1.57079632679 0 1.57079632679
- added joint shoulder_lift_joint: type revolute, parent shoulder_link, child upper_arm_link, origin xyz=0 0 0 rpy=1.570796327 0 0, axis 0 0 1, limit lower=-6.28318530718 upper=6.28318530718 effort=150.0 velocity=3.14159265359
- added joint shoulder_pan_joint: type revolute, parent base_link_inertia, child shoulder_link, origin xyz=0 0 0.089159 rpy=0 0 0, axis 0 0 1, limit lower=-6.28318530718 upper=6.28318530718 effort=150.0 velocity=3.14159265359
- added joint wrist_1_joint: type revolute, parent forearm_link, child wrist_1_link, origin xyz=-0.39225 0 0.10915 rpy=0 0 0, axis 0 0 1, limit lower=-6.28318530718 upper=6.28318530718 effort=28.0 velocity=3.14159265359
- added joint wrist_2_joint: type revolute, parent wrist_1_link, child wrist_2_link, origin xyz=0 -0.09465 -1.9413039509e-11 rpy=1.570796327 0 0, axis 0 0 1, limit lower=-6.28318530718 upper=6.28318530718 effort=28.0 velocity=3.14159265359
- added joint wrist_3-flange: type fixed, parent wrist_3_link, child flange, origin xyz=0 0 0 rpy=0 -1.57079632679 -1.57079632679
- added joint wrist_3_joint: type revolute, parent wrist_2_link, child wrist_3_link, origin xyz=0 0.0823 -1.68800121668e-11 rpy=1.57079632659 3.14159265359 3.14159265359, axis 0 0 1, limit lower=-6.28318530718 upper=6.28318530718 effort=28.0 velocity=3.14159265359
- joint base_joint: origin xyz=0 0 0 rpy=0 0 0 -> xyz=-0.23 -0.1 0.683 rpy=0 0 0; parent base_footprint -> lh_10_body_link

Commit message: Revert "Experiment with removing namespace"
This reverts commit b334f5df1d8d471515a6ba77fdc9beed22ce702e.

File: urdf/little_helper10_arm_on_left.urdf (robot description, URDF)
Before this commit: robot little_helper10, 30 links, 29 joints
Links:
- removed link base
- removed link base_link_inertia
- removed link flange
- removed link forearm_link
- removed link shoulder_link
- removed link tool0
- removed link upper_arm_link
- removed link wrist_1_link
- removed link wrist_2_link
- removed link wrist_3_link
- added link ur5_arm_1_base
- added link ur5_arm_1_base_link
- added link ur5_arm_1_base_link_inertia, mass 4.0; collision mesh filename=package://little_helper_urdf/ur5_to_convert/base.stl; visual mesh filename=package://little_helper_urdf/ur5_to_convert/base.dae
- added link ur5_arm_1_flange
- added link ur5_arm_1_forearm_link, mass 2.275; collision mesh filename=package://little_helper_urdf/ur5_to_convert/forearm.stl; visual mesh filename=package://little_helper_urdf/ur5_to_convert/forearm.dae
- added link ur5_arm_1_shoulder_link, mass 3.7; collision mesh filename=package://little_helper_urdf/ur5_to_convert/shoulder.stl; visual mesh filename=package://little_helper_urdf/ur5_to_convert/shoulder.dae
- added link ur5_arm_1_tool0
- added link ur5_arm_1_upper_arm_link, mass 8.393; collision mesh filename=package://little_helper_urdf/ur5_to_convert/upperarm.stl; visual mesh filename=package://little_helper_urdf/ur5_to_convert/upperarm.dae
- added link ur5_arm_1_wrist_1_link, mass 1.219; collision mesh filename=package://little_helper_urdf/ur5_to_convert/wrist1.stl; visual mesh filename=package://little_helper_urdf/ur5_to_convert/wrist1.dae
- added link ur5_arm_1_wrist_2_link, mass 1.219; collision mesh filename=package://little_helper_urdf/ur5_to_convert/wrist2.stl; visual mesh filename=package://little_helper_urdf/ur5_to_convert/wrist2.dae
- added link ur5_arm_1_wrist_3_link, mass 0.1879; collision mesh filename=package://little_helper_urdf/ur5_to_convert/wrist3.stl; visual mesh filename=package://little_helper_urdf/ur5_to_convert/wrist3.dae
- link base_link: mass None -> 77.0; geometry collision mesh filename=package://little_helper_urdf/mir/collision/mir_100_base.stl; visual mesh filename=package://little_helper_urdf/mir/visual/mir_100_base.stl
Joints:
- removed joint base_link-base_fixed_joint
- removed joint base_link-base_link_inertia
- removed joint elbow_joint
- removed joint flange-tool0
- removed joint shoulder_lift_joint
- removed joint shoulder_pan_joint
- removed joint wrist_1_joint
- removed joint wrist_2_joint
- removed joint wrist_3-flange
- removed joint wrist_3_joint
- added joint ur5_arm_1_base_joint: type fixed, parent lh_10_body_link, child ur5_arm_1_base_link, origin xyz=-0.23 -0.1 0.683 rpy=0 0 0
- added joint ur5_arm_1_base_link-base_fixed_joint: type fixed, parent ur5_arm_1_base_link, child ur5_arm_1_base, origin xyz=0 0 0 rpy=0 0 3.14159265359
- added joint ur5_arm_1_base_link-base_link_inertia: type fixed, parent ur5_arm_1_base_link, child ur5_arm_1_base_link_inertia, origin xyz=0 0 0 rpy=0 0 3.14159265359
- added joint ur5_arm_1_elbow_joint: type revolute, parent ur5_arm_1_upper_arm_link, child ur5_arm_1_forearm_link, origin xyz=-0.425 0 0 rpy=0 0 0, axis 0 0 1, limit lower=-3.14159265359 upper=3.14159265359 effort=150.0 velocity=3.14159265359
- added joint ur5_arm_1_flange-tool0: type fixed, parent ur5_arm_1_flange, child ur5_arm_1_tool0, origin xyz=0 0 0 rpy=1.57079632679 0 1.57079632679
- added joint ur5_arm_1_shoulder_lift_joint: type revolute, parent ur5_arm_1_shoulder_link, child ur5_arm_1_upper_arm_link, origin xyz=0 0 0 rpy=1.570796327 0 0, axis 0 0 1, limit lower=-6.28318530718 upper=6.28318530718 effort=150.0 velocity=3.14159265359
- added joint ur5_arm_1_shoulder_pan_joint: type revolute, parent ur5_arm_1_base_link_inertia, child ur5_arm_1_shoulder_link, origin xyz=0 0 0.089159 rpy=0 0 0, axis 0 0 1, limit lower=-6.28318530718 upper=6.28318530718 effort=150.0 velocity=3.14159265359
- added joint ur5_arm_1_wrist_1_joint: type revolute, parent ur5_arm_1_forearm_link, child ur5_arm_1_wrist_1_link, origin xyz=-0.39225 0 0.10915 rpy=0 0 0, axis 0 0 1, limit lower=-6.28318530718 upper=6.28318530718 effort=28.0 velocity=3.14159265359
- added joint ur5_arm_1_wrist_2_joint: type revolute, parent ur5_arm_1_wrist_1_link, child ur5_arm_1_wrist_2_link, origin xyz=0 -0.09465 -1.9413039509e-11 rpy=1.570796327 0 0, axis 0 0 1, limit lower=-6.28318530718 upper=6.28318530718 effort=28.0 velocity=3.14159265359
- added joint ur5_arm_1_wrist_3-flange: type fixed, parent ur5_arm_1_wrist_3_link, child ur5_arm_1_flange, origin xyz=0 0 0 rpy=0 -1.57079632679 -1.57079632679
- added joint ur5_arm_1_wrist_3_joint: type revolute, parent ur5_arm_1_wrist_2_link, child ur5_arm_1_wrist_3_link, origin xyz=0 0.0823 -1.68800121668e-11 rpy=1.57079632659 3.14159265359 3.14159265359, axis 0 0 1, limit lower=-6.28318530718 upper=6.28318530718 effort=28.0 velocity=3.14159265359
- joint base_joint: origin xyz=-0.23 -0.1 0.683 rpy=0 0 0 -> xyz=0 0 0 rpy=0 0 0; parent lh_10_body_link -> base_footprint

Commit message: Fixed naming

File: urdf/little_helper10_arm_on_left.urdf (robot description, URDF)
Before this commit: robot little_helper10, 30 links, 29 joints
Links:
- added link ur5_base_link
- link base_link: mass None -> 77.0; geometry collision mesh filename=package://little_helper_urdf/mir/collision/mir_100_base.stl; visual mesh filename=package://little_helper_urdf/mir/visual/mir_100_base.stl
Joints:
- added joint ur5_base_joint: type fixed, parent lh_10_body_link, child ur5_base_link, origin xyz=-0.23 -0.1 0.683 rpy=0 0 0
- joint base_joint: origin xyz=-0.23 -0.1 0.683 rpy=0 0 0 -> xyz=0 0 0 rpy=0 0 0; parent lh_10_body_link -> base_footprint
- joint base_link-base_fixed_joint: parent base_link -> ur5_base_link
- joint base_link-base_link_inertia: parent base_link -> ur5_base_link

Commit message: Added virtual laser link and rotated base

File: urdf/little_helper10_arm_on_left.urdf (robot description, URDF)
Before this commit: robot little_helper10, 31 links, 30 joints
Links:
- added link $virtual_laser_link
Joints:
- added joint base_link_to_virtual_laser_joint: type fixed, parent base_link, child virtual_laser_link, origin xyz=0.0 0.0 0.25 rpy=0.0 0.0 0
- joint ur5_base_joint: origin xyz=-0.23 -0.1 0.683 rpy=0 0 0 -> xyz=-0.23 -0.1 0.683 rpy=0 0 -0.785398

Commit message: Update little_helper10_arm_on_left.urdf

File: urdf/little_helper10_arm_on_left.urdf (robot description, URDF)
Before this commit: robot little_helper10, 32 links, 31 joints
Links:
- removed link $virtual_laser_link
- added link virtual_laser_link

Commit message: Added tcp, but without any translation.

File: urdf/little_helper10_arm_on_left.urdf (robot description, URDF)
Before this commit: robot little_helper10, 32 links, 31 joints
Links:
- added link tcp
Joints:
- added joint tool0-tcp: type fixed, parent tool0, child tcp, origin xyz=0 0 0 rpy=0.0 0.0 0.0

Commit message: Added translation

File: urdf/little_helper10_arm_on_left.urdf (robot description, URDF)
Before this commit: robot little_helper10, 33 links, 32 joints
Joints:
- joint tool0-tcp: origin xyz=0 0 0 rpy=0.0 0.0 0.0 -> xyz=0.168 0 0 rpy=0.0 0.0 0.0

Commit message: Fix

File: urdf/little_helper10_arm_on_left.urdf (robot description, URDF)
Before this commit: robot little_helper10, 33 links, 32 joints
Joints:
- joint tool0-tcp: origin xyz=0.168 0 0 rpy=0.0 0.0 0.0 -> xyz=0 0 0.168 rpy=0.0 0.0 0.0
